Commit message: commit before the great change

File: src/atlas_sim/urdf/rover.urdf (robot description, URDF)
Before this commit: robot mock_rover, 6 links, 5 joints
Links:
- link front_left_wheel: geometry collision cylinder length=0.10 radius=0.20; visual cylinder length=0.10 radius=0.20
- link front_right_wheel: geometry collision cylinder length=0.10 radius=0.20; visual cylinder length=0.10 radius=0.20
- link rear_left_wheel: geometry collision cylinder length=0.10 radius=0.20; visual cylinder length=0.10 radius=0.20
- link rear_right_wheel: geometry collision cylinder length=0.10 radius=0.20; visual cylinder length=0.10 radius=0.20

File: src/atlas_sim/urdf/wheels.xacro (robot description, xacro)
@@ -6,6 +6,6 @@
     <origin rpy="1.5708 0 0"/>
     <geometry>
-      <cylinder radius="0.12"
-                length="0.08"/>
+      <cylinder radius="0.20"
+                length="0.10"/>
     </geometry>
   </visual>
@@ -13,6 +13,6 @@
     <origin rpy="1.5708 0 0"/>
     <geometry>
-      <cylinder radius="0.12"
-                length="0.08"/>
+      <cylinder radius="0.20"
+                length="0.10"/>
     </geometry>
   </collision>
